File: Hardware/Schematics/ALU/_autosave-ALU.kicad_sch (KiCad schematic)
At the start: 12 parts

Commit message: Finished Registers, Started ALU
Parts:
- added J? (x4): Conn_01x03, symbol Connector_Generic:Conn_01x03
Connections:
- net Compare/RD != RS: now also J?.1 (Pin_1), J?.3 (Pin_3); no longer U?.8
- net Compare/RD == RS: now also J?.1 (Pin_1), J?.3 (Pin_3); no longer U?.12
- net GND: now also U?.7 (GND), U?.7 (GND)
- net VCC: now also U?.14 (VCC), U?.14 (VCC)
- net at U?.10, U?.11: now also J?.1 (Pin_1)
- net at U?.13, U?.9: now also J?.3 (Pin_3)
- net at U?.3, U?.4: now also J?.3 (Pin_3)
- net at U?.1, U?.5: now also J?.1 (Pin_1)
- net at U?.8: now also J?.7 (Pin_7)
- net at J?.3 (Pin_3): now also U?.2
- new net: J?.2 (Pin_2), U?.8
- new net: J?.2 (Pin_2), U?.12
