File: Hardware/Schematics/ALU/ALU.kicad_sch (KiCad schematic)
At the start: 12 parts

Commit message: ALU Design Finished
Parts:
- removed U? (x8): 74LS02, symbol 74xx:74LS02
- added C1, C10, C11, C12, C13, C14, C15, C16, C17, C18, C19, C2, C20, C21, C22, C3, C4, C5, C6, C7, C8, C9: C, Capacitor_THT:C_Rect_L9.0mm_W2.5mm_P7.50mm_MKT, symbol Device:C
- added J5: Conn_02x05_Counter_Clockwise, Connector_PinHeader_2.54mm:PinHeader_2x05_P2.54mm_Horizontal, symbol Connector_Generic:Conn_02x05_Counter_Clockwise
- added U1, U3: 74LS113, Package_DIP:DIP-14_W7.62mm_Socket_LongPads, symbol 74xx:74LS113
- added U2: 74LS32, Package_DIP:DIP-14_W7.62mm_Socket_LongPads, symbol 74xx:74LS32
- added U22: 74LS08, Package_DIP:DIP-14_W7.62mm_Socket_LongPads, symbol 74xx:74LS08
- J1, J2, J4: renamed from J?; footprint (none) -> Connector_PinHeader_2.54mm:PinHeader_1x10_P2.54mm_Horizontal
- J3: renamed from J?; footprint (none) -> Connector_PinHeader_2.54mm:PinHeader_2x05_P2.54mm_Horizontal
Connections:
- net Compare/Res_{1} is gone; now on net Adder/Out_{1}: J4.3 (Pin_3)
- net Adder/C_{Flag}: now also U1.11 (J)
- net Adder/C_{Out}: now also U1.3 (J)
- net Compare/RD != RS: now also U2.2
- net Compare/RD == RS: now also U2.5
- net GND: now also C1.2, C10.2, C11.2, C12.2, C13.2, C14.2, C15.2, C16.2, C17.2, C18.2, C19.2, C2.2, C20.2, C21.2, C22.2, C3.2, C4.2, C5.2, C6.2, C7.2, C8.2, C9.2, J5.6 (Pin_6), U1.7 (GND), U2.7 (GND), U22.7 (GND), U3.11 (J), U3.12 (K), U3.7 (GND)
- net VCC: now also C1.1, C10.1, C11.1, C12.1, C13.1, C14.1, C15.1, C16.1, C17.1, C18.1, C19.1, C2.1, C20.1, C21.1, C22.1, C3.1, C4.1, C5.1, C6.1, C7.1, C8.1, C9.1, J5.1 (Pin_1), U1.10 (~{S}), U1.14 (VCC), U1.4 (~{S}), U2.14 (VCC), U22.14 (VCC), U3.10 (~{S}), U3.14 (VCC), U3.4 (~{S})
- net at J3.3 (Pin_3): now also U22.2
- net at J3.7 (Pin_7): now also U22.1
- new net: J5.3 (Pin_3), U2.4
- new net: U2.6, U3.2 (K)
- new net: J5.5 (Pin_5), U1.2 (K)
- new net: J5.7 (Pin_7), U1.5 (Q)
- new net: J5.2 (Pin_2), U2.1
- new net: U2.3, U3.3 (J)
- new net: J5.9 (Pin_9), U3.5 (Q)
- new net: J5.10 (Pin_10), U3.6 (~{Q})
- new net: J5.4 (Pin_4), U1.12 (K)
- new net: J5.8 (Pin_8), U1.9 (Q)
- new net CLK: U1.1 (C), U1.13 (C), U22.3, U3.1 (C), U3.13 (C)
