File: Hardware/Schematics/ALU/Adder.kicad_sch (KiCad schematic)
At the start: 22 parts

Commit message: ALU Design Finished
Parts:
- removed U?: 74LS32, symbol 74xx:74LS32
- U10, U11: renamed from U?; footprint (none) -> Package_DIP:DIP-16_W7.62mm_Socket_LongPads
- U12, U8, U9: renamed from U?; footprint (none) -> Package_DIP:DIP-20_W7.62mm_Socket_LongPads
- U4, U5, U6, U7: renamed from U?; footprint (none) -> Package_DIP:DIP-14_W7.62mm_Socket_LongPads
Connections:
- net RD_{4}: now also U11.10 (A1); no longer U11.1 (A4)
- net RD_{5}: now also U11.8 (A2); no longer U11.3 (A3)
- net RD_{6}: now also U11.3 (A3); no longer U11.8 (A2)
- net RD_{7}: now also U11.1 (A4); no longer U11.10 (A1)
