File: Hardware/Schematics/ALU/Compare.kicad_sch (KiCad schematic)
At the start: 22 parts

Commit message: Finished Registers, Started ALU
Parts:
- removed U? (x3): 74LS245, symbol 74xx:74LS245
- removed U? (x5): 74LS04, symbol 74xx:74LS04
- removed U? (x10): 74LS86, symbol 74xx:74LS86
- removed U? (x2): 74LS83, symbol 74xx:74LS83
- removed U? (x2): 74LS32, symbol 74xx:74LS32
- added RN?: R_Network08, Resistor_THT:R_Array_SIP9, symbol Device:R_Network08
- added U? (x9): 74LS32, symbol 74xx:74LS32
- added U? (x10): 74LS86, symbol 74xx:74LS86
- added U? (x2): 74LS04, symbol 74xx:74LS04
- added U? (x3): 74LS245, symbol 74xx:74LS245
Connections:
- net GND: now also RN?.1 (common), U?.10 (GND), U?.10 (GND), U?.10 (GND), U?.7 (GND), U?.7 (GND), U?.7 (GND), U?.7 (GND)
- net RD_{0}: now also U?.2 (A0)
- net RD_{1}: now also U?.3 (A1)
- net RD_{2}: now also U?.4 (A2)
- net RD_{3}: now also U?.5 (A3)
- net RD_{4}: now also U?.6 (A4)
- net RD_{5}: now also U?.7 (A5)
- net RD_{6}: now also U?.8 (A6)
- net RD_{7}: now also U?.9 (A7)
- net RS_{0}: now also U?.2 (A0)
- net RS_{1}: now also U?.3 (A1)
- net RS_{2}: now also U?.4 (A2)
- net RS_{3}: now also U?.5 (A3)
- net RS_{4}: now also U?.6 (A4)
- net RS_{5}: now also U?.7 (A5)
- net RS_{6}: now also U?.8 (A6)
- net RS_{7}: now also U?.9 (A7)
- net VCC: now also U?.1 (A->B), U?.1 (A->B), U?.1 (A->B), U?.14 (VCC), U?.14 (VCC), U?.14 (VCC), U?.14 (VCC), U?.20 (VCC), U?.20 (VCC), U?.20 (VCC)
- new net: U?.1, U?.3 (x2)
- new net: U?.2, U?.6 (x2)
- new net: U?.10, U?.6 (x2)
- new net: U?.4, U?.8 (x2)
- new net: U?.3, U?.9 (x2)
- new net: RN?.7 (R6), U?.10, U?.16 (B2)
- new net: U?.16 (B2), U?.16 (B2), U?.9
- new net: U?.11, U?.5 (x2)
- new net: RN?.2 (R1), U?.11 (B7), U?.13
- new net: RN?.3 (R2), U?.10, U?.12 (B6)
- new net: RN?.4 (R3), U?.13 (B5), U?.5
- new net: RN?.5 (R4), U?.14 (B4), U?.2
- new net: RN?.6 (R5), U?.13, U?.15 (B3)
- new net: RN?.8 (R7), U?.17 (B1), U?.5
- new net: RN?.9 (R8), U?.18 (B0), U?.2
- new net: U?.13 (B5), U?.13 (B5), U?.4
- new net: U?.19 (CE), U?.6
- new net: U?.1, U?.18 (B0), U?.18 (B0)
- new net: U?.17 (B1), U?.17 (B1), U?.4
- new net: U?.12, U?.8
- new net: U?.11, U?.13
- new net: U?.11 (B7), U?.11 (B7), U?.12
- new net: U?.12 (B6), U?.12 (B6), U?.9
- new net: U?.1, U?.14 (B4), U?.14 (B4)
- new net: U?.12, U?.15 (B3), U?.15 (B3)
- new net RD != RS: U?.3, U?.8
- new net RD == RS: U?.4
- new net Res_{0}: U?.2 (A0)
- new net Res_{1}: U?.3 (A1)
- new net Res_{2}: U?.4 (A2)
- new net Res_{3}: U?.5 (A3)
- new net Res_{4}: U?.6 (A4)
- new net Res_{5}: U?.7 (A5)
- new net Res_{6}: U?.8 (A6)
- new net Res_{7}: U?.9 (A7)
- new net ~{CMP}: U?.19 (CE), U?.19 (CE), U?.5

Commit message: ALU Design Finished
Parts:
- removed U?: 74LS32, symbol 74xx:74LS32
- U16, U17, U18: renamed from U?; footprint (none) -> Package_DIP:DIP-20_W7.62mm_Socket_LongPads
- U19, U20, U21, U5, U7: renamed from U?; footprint (none) -> Package_DIP:DIP-14_W7.62mm_Socket_LongPads
- gave numbers to parts that had none: 1
