File: Hardware/Schematics/ALU/NAND.kicad_sch (KiCad schematic)
At the start: 11 parts

Commit message: ALU Design Finished
Parts:
- U13, U14: renamed from U?; footprint (none) -> Package_DIP:DIP-14_W7.62mm_Socket_LongPads
- U15: renamed from U?; footprint (none) -> Package_DIP:DIP-20_W7.62mm_Socket_LongPads
Changed lines of the file:
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@@
   (symbol (lib_id "74xx:74LS00") (at 80.264 75.057 0) (unit 3)
     (in_bom yes) (on_board yes) (fields_autoplaced)
-    (property "Reference" "U?" (id 0) (at 80.264 66.04 0))
+    (property "Reference" "U14" (id 0) (at 80.264 66.04 0))
     (property "Value" "74LS00" (id 1) (at 80.264 68.58 0))
-    (property "Footprint" "" (id 2) (at 80.264 75.057 0)
+    (property "Footprint" "Package_DIP:DIP-14_W7.62mm_Socket_LongPads" (id 2) (at 80.264 75.057 0)
       (effects (font (size 1.27 1.27)) hide)
     )
@@
   (symbol (lib_id "74xx:74LS00") (at 80.264 82.677 0) (unit 4)
     (in_bom yes) (on_board yes) (fields_autoplaced)
-    (property "Reference" "U?" (id 0) (at 80.264 73.66 0))
+    (property "Reference" "U14" (id 0) (at 80.264 73.66 0))
     (property "Value" "74LS00" (id 1) (at 80.264 76.2 0))
-    (property "Footprint" "" (id 2) (at 80.264 82.677 0)
+    (property "Footprint" "Package_DIP:DIP-14_W7.62mm_Socket_LongPads" (id 2) (at 80.264 82.677 0)
       (effects (font (size 1.27 1.27)) hide)
     )
@@
   (symbol (lib_id "74xx:74LS00") (at 33.782 69.723 0) (unit 5)
     (in_bom yes) (on_board yes) (fields_autoplaced)
-    (property "Reference" "U?" (id 0) (at 40.64 68.4529 0)
+    (property "Reference" "U13" (id 0) (at 40.64 68.4529 0)
       (effects (font (size 1.27 1.27)) (justify left))
     )
@@
       (effects (font (size 1.27 1.27)) (justify left))
     )
-    (property "Footprint" "" (id 2) (at 33.782 69.723 0)
+    (property "Footprint" "Package_DIP:DIP-14_W7.62mm_Socket_LongPads" (id 2) (at 33.782 69.723 0)
       (effects (font (size 1.27 1.27)) hide)
     )
@@
   (symbol (lib_id "74xx:74LS00") (at 80.264 44.577 0) (unit 3)
     (in_bom yes) (on_board yes) (fields_autoplaced)
-    (property "Reference" "U?" (id 0) (at 80.264 35.687 0))
+    (property "Reference" "U13" (id 0) (at 80.264 35.687 0))
     (property "Value" "74LS00" (id 1) (at 80.264 38.227 0))
-    (property "Footprint" "" (id 2) (at 80.264 44.577 0)
+    (property "Footprint" "Package_DIP:DIP-14_W7.62mm_Socket_LongPads" (id 2) (at 80.264 44.577 0)
       (effects (font (size 1.27 1.27)) hide)
     )
@@
   (symbol (lib_id "74xx:74LS00") (at 80.264 59.817 0) (unit 1)
     (in_bom yes) (on_board yes) (fields_autoplaced)
-    (property "Reference" "U?" (id 0) (at 80.264 50.8 0))
+    (property "Reference" "U14" (id 0) (at 80.264 50.8 0))
     (property "Value" "74LS00" (id 1) (at 80.264 53.34 0))
-    (property "Footprint" "" (id 2) (at 80.264 59.817 0)
+    (property "Footprint" "Package_DIP:DIP-14_W7.62mm_Socket_LongPads" (id 2) (at 80.264 59.817 0)
       (effects (font (size 1.27 1.27)) hide)
     )
@@
   (symbol (lib_id "power:VCC") (at 121.539 21.717 0) (unit 1)
     (in_bom yes) (on_board yes) (fields_autoplaced)
-    (property "Reference" "#PWR?" (id 0) (at 121.539 25.527 0)
+    (property "Reference" "#PWR032" (id 0) (at 121.539 25.527 0)
       (effects (font (size 1.27 1.27)) hide)
     )
@@
   (symbol (lib_id "74xx:74LS245") (at 126.111 42.037 0) (unit 1)
     (in_bom yes) (on_board yes) (fields_autoplaced)
-    (property "Reference" "U?" (id 0) (at 128.1304 21.971 0)
+    (property "Reference" "U15" (id 0) (at 128.1304 21.971 0)
       (effects (font (size 1.27 1.27)) (justify left))
     )
@@
       (effects (font (size 1.27 1.27)) (justify left))
     )
-    (property "Footprint" "" (id 2) (at 126.111 42.037 0)
+    (property "Footprint" "Package_DIP:DIP-20_W7.62mm_Socket_LongPads" (id 2) (at 126.111 42.037 0)
       (effects (font (size 1.27 1.27)) hide)
     )
@@
   (symbol (lib_id "power:VCC") (at 33.782 57.023 0) (unit 1)
     (in_bom yes) (on_board yes) (fields_autoplaced)
-    (property "Reference" "#PWR?" (id 0) (at 33.782 60.833 0)
+    (property "Reference" "#PWR028" (id 0) (at 33.782 60.833 0)
       (effects (font (size 1.27 1.27)) hide)
     )
@@
   (symbol (lib_id "74xx:74LS00") (at 80.264 29.337 0) (unit 1)
     (in_bom yes) (on_board yes) (fields_autoplaced)
-    (property "Reference" "U?" (id 0) (at 80.264 20.32 0))
+    (property "Reference" "U13" (id 0) (at 80.264 20.32 0))
     (property "Value" "74LS00" (id 1) (at 80.264 22.86 0))
-    (property "Footprint" "" (id 2) (at 80.264 29.337 0)
+    (property "Footprint" "Package_DIP:DIP-14_W7.62mm_Socket_LongPads" (id 2) (at 80.264 29.337 0)
       (effects (font (size 1.27 1.27)) hide)
     )
@@
   (symbol (lib_id "power:VCC") (at 43.942 57.023 0) (unit 1)
     (in_bom yes) (on_board yes) (fields_autoplaced)
-    (property "Reference" "#PWR?" (id 0) (at 43.942 60.833 0)
+    (property "Reference" "#PWR030" (id 0) (at 43.942 60.833 0)
       (effects (font (size 1.27 1.27)) hide)
     )
@@
   (symbol (lib_id "power:GND") (at 43.942 82.423 0) (unit 1)
     (in_bom yes) (on_board yes) (fields_autoplaced)
-    (property "Reference" "#PWR?" (id 0) (at 43.942 88.773 0)
+    (property "Reference" "#PWR031" (id 0) (at 43.942 88.773 0)
       (effects (font (size 1.27 1.27)) hide)
     )
@@
   (symbol (lib_id "74xx:74LS00") (at 80.264 36.957 0) (unit 2)
     (in_bom yes) (on_board yes) (fields_autoplaced)
-    (property "Reference" "U?" (id 0) (at 80.264 27.94 0))
+    (property "Reference" "U13" (id 0) (at 80.264 27.94 0))
     (property "Value" "74LS00" (id 1) (at 80.264 30.48 0))
-    (property "Footprint" "" (id 2) (at 80.264 36.957 0)
+    (property "Footprint" "Package_DIP:DIP-14_W7.62mm_Socket_LongPads" (id 2) (at 80.264 36.957 0)
       (effects (font (size 1.27 1.27)) hide)
     )
@@
   (symbol (lib_id "74xx:74LS00") (at 80.264 67.437 0) (unit 2)
     (in_bom yes) (on_board yes) (fields_autoplaced)
-    (property "Reference" "U?" (id 0) (at 80.264 58.42 0))
+    (property "Reference" "U14" (id 0) (at 80.264 58.42 0))
     (property "Value" "74LS00" (id 1) (at 80.264 60.96 0))
-    (property "Footprint" "" (id 2) (at 80.264 67.437 0)
+    (property "Footprint" "Package_DIP:DIP-14_W7.62mm_Socket_LongPads" (id 2) (at 80.264 67.437 0)
       (effects (font (size 1.27 1.27)) hide)
     )
@@
   (symbol (lib_id "power:GND") (at 126.111 62.357 0) (unit 1)
     (in_bom yes) (on_board yes) (fields_autoplaced)
-    (property "Reference" "#PWR?" (id 0) (at 126.111 68.707 0)
+    (property "Reference" "#PWR033" (id 0) (at 126.111 68.707 0)
       (effects (font (size 1.27 1.27)) hide)
     )
@@
   (symbol (lib_id "74xx:74LS00") (at 80.264 52.197 0) (unit 4)
     (in_bom yes) (on_board yes) (fields_autoplaced)
-    (property "Reference" "U?" (id 0) (at 80.264 43.18 0))
+    (property "Reference" "U13" (id 0) (at 80.264 43.18 0))
     (property "Value" "74LS00" (id 1) (at 80.264 45.72 0))
-    (property "Footprint" "" (id 2) (at 80.264 52.197 0)
+    (property "Footprint" "Package_DIP:DIP-14_W7.62mm_Socket_LongPads" (id 2) (at 80.264 52.197 0)
       (effects (font (size 1.27 1.27)) hide)
     )
@@
   (symbol (lib_id "74xx:74LS00") (at 43.942 69.723 0) (unit 5)
     (in_bom yes) (on_board yes) (fields_autoplaced)
-    (property "Reference" "U?" (id 0) (at 50.8 68.4529 0)
+    (property "Reference" "U14" (id 0) (at 50.8 68.4529 0)
       (effects (font (size 1.27 1.27)) (justify left))
     )
@@
       (effects (font (size 1.27 1.27)) (justify left))
     )
-    (property "Footprint" "" (id 2) (at 43.942 69.723 0)
+    (property "Footprint" "Package_DIP:DIP-14_W7.62mm_Socket_LongPads" (id 2) (at 43.942 69.723 0)
       (effects (font (size 1.27 1.27)) hide)
     )
@@
   (symbol (lib_id "power:GND") (at 33.782 82.423 0) (unit 1)
     (in_bom yes) (on_board yes) (fields_autoplaced)
-    (property "Reference" "#PWR?" (id 0) (at 33.782 88.773 0)
-      (effects (font (size 1.27 1.27)) hide)
-    )
+    (property "Reference" "#PWR029" (id 0) (at 33.782 88.773 0)
+      (effects (font (size 1.27 1.27)) hide)
+    )
