File: Hardware/Schematics/Datapath_Controller/Datapath_Controller.kicad_pcb (KiCad board)
At the start: 2 copper layers, 4 parts

Commit message: Finished Datapath Controller
Parts:
- removed the REF** at (197.3, 144.6)
- removed the REF** at (197.3, 21.2)
- removed the REF** at (23.3, 21.2)
- removed the REF** at (23.3, 144.6)
- added ?: , , F.Cu at (40.0, 191.8)
- added C1: C, Capacitor_THT:C_Rect_L7.0mm_W2.5mm_P5.00mm, F.Cu at (214.9, 72.7)
- added C2: C, Capacitor_THT:C_Rect_L7.0mm_W2.5mm_P5.00mm, F.Cu at (110.4, 86.5)
- added C3: C, Capacitor_THT:C_Rect_L7.0mm_W2.5mm_P5.00mm, F.Cu at (92.4, 63.7)
- added C4: C, Capacitor_THT:C_Rect_L7.0mm_W2.5mm_P5.00mm, F.Cu at (214.9, 51.2)
- added C5: C, Capacitor_THT:C_Rect_L7.0mm_W2.5mm_P5.00mm, F.Cu at (92.1, 79.8)
- added C6: C, Capacitor_THT:C_Rect_L7.0mm_W2.5mm_P5.00mm, F.Cu at (215.2, 91.5)
- added J1: Conn_01x10, Connector_PinHeader_2.54mm:PinHeader_1x10_P2.54mm_Vertical, F.Cu at (174.4, 90.9)
- added J10: Conn_01x10, Connector_PinHeader_2.54mm:PinHeader_1x10_P2.54mm_Vertical, F.Cu at (241.0, 110.0)
- added J2: Conn_01x10, Connector_PinHeader_2.54mm:PinHeader_1x10_P2.54mm_Vertical, F.Cu at (111.6, 27.6)
- added J3: Conn_02x05_Counter_Clockwise, Connector_PinHeader_2.54mm:PinHeader_2x05_P2.54mm_Vertical, F.Cu at (163.9, 145.5)
- added J4: Conn_01x10, Connector_PinHeader_2.54mm:PinHeader_1x10_P2.54mm_Vertical, F.Cu at (144.4, 27.4)
- added J5: Conn_02x05_Counter_Clockwise, Connector_PinHeader_2.54mm:PinHeader_2x05_P2.54mm_Vertical, F.Cu at (162.6, 82.1)
- added J6: Conn_01x08, Connector_PinHeader_2.54mm:PinHeader_1x10_P2.54mm_Vertical, F.Cu at (281.2, 42.4)
- added J7: Conn_01x08, Connector_PinHeader_2.54mm:PinHeader_1x10_P2.54mm_Vertical, F.Cu at (174.4, 34.3)
- added J8: Conn_01x08, Connector_PinHeader_2.54mm:PinHeader_1x10_P2.54mm_Vertical, F.Cu at (165.2, 120.4)
- added J9: Conn_01x19, Connector_PinHeader_2.54mm:PinHeader_1x19_P2.54mm_Vertical, F.Cu at (271.8, 17.5)
- added REF**: MountingHole_5.3mm_M5, MountingHole:MountingHole_5.3mm_M5, F.Cu at (40.0, 191.8)
- added REF**: MountingHole_5.3mm_M5, MountingHole:MountingHole_5.3mm_M5, F.Cu at (163.4, 17.8)
- added REF**: MountingHole_5.3mm_M5, MountingHole:MountingHole_5.3mm_M5, F.Cu at (40.0, 17.8)
- added REF**: MountingHole_5.5mm, MountingHole:MountingHole_5.5mm, F.Cu at (270.6, 180.8)
- added REF**: MountingHole_5.5mm, MountingHole:MountingHole_5.5mm, F.Cu at (195.8, 162.4)
- added REF**: MountingHole_5.3mm_M5, MountingHole:MountingHole_5.3mm_M5, F.Cu at (163.4, 191.8)
- added U1: 74LS04, Package_DIP:DIP-14_W7.62mm_Socket_LongPads, F.Cu at (103.9, 91.2)
- added U2: 74LS245, Package_DIP:DIP-20_W7.62mm_Socket_LongPads, F.Cu at (120.2, 73.0)
- added U3: 74LS245, Package_DIP:DIP-20_W7.62mm_Socket_LongPads, F.Cu at (120.2, 57.1)
- added U4: 28C16, Package_DIP:DIP-24_W15.24mm_Socket_LongPads, F.Cu at (220.3, 55.7)
- added U5: 28C16, Package_DIP:DIP-24_W15.24mm_Socket_LongPads, F.Cu at (220.3, 76.3)
- added U6: 28C16, Package_DIP:DIP-24_W15.24mm_Socket_LongPads, F.Cu at (220.3, 96.8)
Routing:
- net GND: track 0.00 -> 650.4 mm
- net VCC: track 0.00 -> 576.8 mm, vias 0 -> 1
- net Net-(U5-Pad17): track 0.00 -> 308.8 mm, vias 0 -> 1
- net Net-(J6-Pad2): track 0.00 -> 293.6 mm
- net Net-(J6-Pad3): track 0.00 -> 289.3 mm
- net Net-(J6-Pad4): track 0.00 -> 285.4 mm
- net Net-(J6-Pad5): track 0.00 -> 279.0 mm
- net Net-(J6-Pad6): track 0.00 -> 274.4 mm
- net Net-(J6-Pad7): track 0.00 -> 269.1 mm
- net Net-(J6-Pad8): track 0.00 -> 264.5 mm
- net Net-(J6-Pad9): track 0.00 -> 259.1 mm
- net Net-(J3-Pad8): track 0.00 -> 221.6 mm, vias 0 -> 1
- net Net-(J3-Pad7): track 0.00 -> 208.9 mm, vias 0 -> 1
- net Net-(J3-Pad9): track 0.00 -> 206.5 mm, vias 0 -> 3
- net Net-(J3-Pad2): track 0.00 -> 170.3 mm, vias 0 -> 2
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- added copper zone on B.Cu, net GND
- added copper zone on F.Cu, net GND
