File: Hardware/Schematics/ControlUnit/ControlUnit.kicad_sch (KiCad schematic)
At the start: 9 parts

Commit message: Interim
Parts:
- added D? (x4): LED, LED_THT:LED_D3.0mm, symbol Device:LED
- added R?: R, symbol Device:R
Connections:
- net GND: now also R?.2
- net wb0: no longer U?.10 (A0), U?.10 (A0)
- net wb1: no longer U?.9 (A1), U?.9 (A1)
- net wb2: no longer U?.8 (A2), U?.8 (A2)
- net wb3: no longer U?.7 (A3), U?.7 (A3)
- net wb4: no longer U?.6 (A4), U?.6 (A4)
- net wb5: no longer U?.5 (A5), U?.5 (A5)
- net wb6: no longer U?.4 (A6), U?.4 (A6)
- net wb7: no longer U?.3 (A7), U?.3 (A7)
- net at U?.1 (~{MR}): now also U?.11 (D0)
- net at U?.11 (Q3): now also U?.1 (A14), U?.1 (A14), U?.1 (A14)
- net at U?.12 (Q2): now also U?.26 (A13), U?.26 (A13), U?.26 (A13)
- net INS_0: now reaches U?.10 (A0)
- net INS_0: now also U?.10 (A0), U?.10 (A0)
- net at U?.2 (A12): now also U?.13 (Q1), U?.2 (A12), U?.2 (A12)
- net at U?.23 (A11): now also U?.14 (Q0), U?.23 (A11), U?.23 (A11)
- net INS_7: now reaches U?.3 (A7)
- net INS_7: now also U?.3 (A7), U?.3 (A7)
- net INS_6: now reaches U?.4 (A6)
- net INS_6: now also U?.4 (A6), U?.4 (A6)
- net INS_5: now reaches U?.5 (A5)
- net INS_5: now also U?.5 (A5), U?.5 (A5)
- net INS_4: now reaches U?.6 (A4)
- net INS_4: now also U?.6 (A4), U?.6 (A4)
- net INS_3: now reaches U?.7 (A3)
- net INS_3: now also U?.7 (A3), U?.7 (A3)
- net INS_2: now reaches U?.8 (A2)
- net INS_2: now also U?.8 (A2), U?.8 (A2)
- net INS_1: now reaches U?.9 (A1)
- net INS_1: now also U?.9 (A1), U?.9 (A1)
- net at U?.12 (D1): now also D?.2 (A)
- net at U?.13 (D2): now also D?.2 (A)
- net at U?.15 (D3): now also D?.2 (A)
- net at U?.16 (D4): now also D?.2 (A)
- new net: D?.1 (K), D?.1 (K), D?.1 (K), D?.1 (K), R?.1

Commit message: Boards Done
Parts:
- removed J?: Conn_01x05, Connector_PinHeader_2.54mm:PinHeader_1x05_P2.54mm_Vertical, symbol Connector_Generic:Conn_01x05
- removed U? (x3): 74LS109, symbol 74xx:74LS109
- added J1: Conn_01x06, Connector_PinSocket_2.54mm:PinSocket_1x06_P2.54mm_Vertical, symbol Connector_Generic:Conn_01x06
- added J3, J7, J8: Conn_01x08_Female, Connector_PinSocket_2.54mm:PinSocket_1x08_P2.54mm_Vertical, symbol Connector:Conn_01x08_Female
- added J4: Conn_02x05_Counter_Clockwise, Connector_PinHeader_2.54mm:PinHeader_2x05_P2.54mm_Vertical, symbol Connector_Generic:Conn_02x05_Counter_Clockwise
- added J5: Conn_01x10, Connector_PinHeader_2.54mm:PinHeader_1x10_P2.54mm_Vertical, symbol Connector_Generic:Conn_01x10
- added J6: Conn_01x18, Connector_PinSocket_2.54mm:PinSocket_1x18_P2.54mm_Vertical, symbol Connector_Generic:Conn_01x18
- added J9: Conn_01x01_Female, Connector_PinSocket_2.54mm:PinSocket_1x01_P2.54mm_Horizontal, symbol Connector:Conn_01x01_Female
- added U6, U7: 28C256, Package_DIP:DIP-28_W15.24mm_Socket_LongPads, symbol Memory_EEPROM:28C256
- R1: renamed from R?; footprint (none) -> Resistor_THT:R_Axial_DIN0204_L3.6mm_D1.6mm_P2.54mm_Vertical
- U2: renamed from U?; footprint (none) -> Package_DIP:DIP-16_W7.62mm_Socket_LongPads
- U3, U4, U5: renamed from U?; footprint (none) -> Package_DIP:DIP-28_W15.24mm_Socket_LongPads
- gave numbers to parts that had none: 5
Connections:
- net GND: now also U3.14 (GND), U3.20 (~{CS}), U3.21 (A10), U3.22 (~{OE}), U3.24 (A9), U3.25 (A8), U4.14 (GND), U4.20 (~{CS}), U4.21 (A10), U4.22 (~{OE}), U4.24 (A9), U4.25 (A8), U5.14 (GND), U5.20 (~{CS}), U5.21 (A10), U5.22 (~{OE}), U5.24 (A9), U5.25 (A8), J1.6 (Pin_6), J4.6 (Pin_6), J5.1 (Pin_1), J6.18 (Pin_18), U6.14 (GND), U6.20 (~{CS}), U6.21 (A10), U6.22 (~{OE}), U6.24 (A9), U6.25 (A8), U7.14 (GND), U7.20 (~{CS}), U7.21 (A10), U7.22 (~{OE}), U7.24 (A9), U7.25 (A8)
- net INS_0: now also U6.10 (A0), U7.10 (A0)
- net INS_1: now also U6.9 (A1), U7.9 (A1)
- net INS_2: now also U6.8 (A2), U7.8 (A2)
- net INS_3: now also U6.7 (A3), U7.7 (A3)
- net INS_4: now also U6.6 (A4), U7.6 (A4)
- net INS_5: now also U6.5 (A5), U7.5 (A5)
- net INS_6: now also U6.4 (A6), U7.4 (A6)
- net INS_7: now also U6.3 (A7), U7.3 (A7)
- net Instruction Data/NextINS: now also J9.1 (Pin_1)
- net VCC: now also U3.28 (VCC), U4.28 (VCC), U5.28 (VCC), J1.1 (Pin_1), J4.1 (Pin_1), J5.10 (Pin_10), J6.1 (Pin_1), U6.28 (VCC), U7.28 (VCC)
- net rd: now also J1.4 (Pin_4)
- net wr: now also J1.3 (Pin_3)
- net A14: now reaches U2.11 (Q3), U3.1 (A14), U4.1 (A14), U5.1 (A14)
- net A14: now also U6.1 (A14), U7.1 (A14)
- net A13: now reaches U2.12 (Q2), U3.26 (A13), U4.26 (A13), U5.26 (A13)
- net A13: now also U6.26 (A13), U7.26 (A13)
- net A12: now reaches U2.13 (Q1), U3.2 (A12), U4.2 (A12), U5.2 (A12)
- net A12: now also U6.2 (A12), U7.2 (A12)
- net A11: now reaches U2.14 (Q0), U3.23 (A11), U4.23 (A11), U5.23 (A11)
- net A11: now also U6.23 (A11), U7.23 (A11)
- net at U2.2 (CP): now also J1.2 (Pin_2)
- net at U3.11 (D0): now also J4.2 (Pin_2)
- net at U3.12 (D1): now also J4.3 (Pin_3)
- net at U3.13 (D2): now also J4.4 (Pin_4)
- net at U3.15 (D3): now also J4.7 (Pin_7)
- net at U3.16 (D4): now also J4.8 (Pin_8)
- net at U3.17 (D5): now also J4.9 (Pin_9)
- net at U3.18 (D6): now also J4.10 (Pin_10)
- net at U5.11 (D0): now also J3.1 (Pin_1)
- net at U5.12 (D1): now also J3.2 (Pin_2)
- net at U5.13 (D2): now also J3.3 (Pin_3)
- net at U5.15 (D3): now also J3.4 (Pin_4)
- net at U5.16 (D4): now also J3.5 (Pin_5)
- net at U5.17 (D5): now also J3.6 (Pin_6)
- net at U5.18 (D6): now also J3.7 (Pin_7)
- net at U5.19 (D7): now also J3.8 (Pin_8)
- new net: J8.1 (Pin_1), U7.11 (D0)
- new net: J8.2 (Pin_2), U7.12 (D1)
- new net: J8.3 (Pin_3), U7.13 (D2)
- new net: J8.4 (Pin_4), U7.15 (D3)
- new net: J8.5 (Pin_5), U7.16 (D4)
- new net: J8.6 (Pin_6), U7.17 (D5)
- new net: J8.7 (Pin_7), U7.18 (D6)
- new net: J8.8 (Pin_8), U7.19 (D7)
- new net: J7.1 (Pin_1), U6.11 (D0)
- new net: J7.2 (Pin_2), U6.12 (D1)
- new net: J7.3 (Pin_3), U6.13 (D2)
- new net: J7.4 (Pin_4), U6.15 (D3)
- new net: J7.5 (Pin_5), U6.16 (D4)
- new net: J7.6 (Pin_6), U6.17 (D5)
- new net: J7.7 (Pin_7), U6.18 (D6)
- new net: J7.8 (Pin_8), U6.19 (D7)
- new net CLK: J1.5 (Pin_5), J4.5 (Pin_5)
- new net OP_0: J5.9 (Pin_9), J6.2 (Pin_2)
- new net OP_1: J5.8 (Pin_8), J6.3 (Pin_3)
- new net OP_10: J6.12 (Pin_12)
- new net OP_11: J6.13 (Pin_13)
- new net OP_12: J6.14 (Pin_14)
- new net OP_13: J6.15 (Pin_15)
- new net OP_14: J6.16 (Pin_16)
- new net OP_15: J6.17 (Pin_17)
- new net OP_2: J5.7 (Pin_7), J6.4 (Pin_4)
- new net OP_3: J5.6 (Pin_6), J6.5 (Pin_5)
- new net OP_4: J5.5 (Pin_5), J6.6 (Pin_6)
- new net OP_5: J5.4 (Pin_4), J6.7 (Pin_7)
- new net OP_6: J5.3 (Pin_3), J6.8 (Pin_8)
- new net OP_7: J5.2 (Pin_2), J6.9 (Pin_9)
- new net OP_8: J6.10 (Pin_10)
- new net OP_9: J6.11 (Pin_11)
