File: Hardware/Schematics/ControlUnit/InsData.kicad_sch (KiCad schematic)
At the start: 5 parts

Commit message: Boards Done
Parts:
- U10, U11, U9: renamed from U?; footprint (none) -> Package_DIP:DIP-20_W7.62mm_Socket_LongPads
- U8: renamed from U?; footprint (none) -> Package_DIP:DIP-16_W7.62mm_Socket_LongPads
Changed lines of the file:
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@@
   (symbol (lib_id "power:GND") (at 41.656 94.996 0) (unit 1)
     (in_bom yes) (on_board yes) (fields_autoplaced)
-    (property "Reference" "#PWR?" (id 0) (at 41.656 101.346 0)
+    (property "Reference" "#PWR0124" (id 0) (at 41.656 101.346 0)
       (effects (font (size 1.27 1.27)) hide)
     )
@@
   (symbol (lib_id "74xx:74LS377") (at 99.822 132.08 0) (unit 1)
     (in_bom yes) (on_board yes) (fields_autoplaced)
-    (property "Reference" "U?" (id 0) (at 101.8414 112.014 0)
+    (property "Reference" "U11" (id 0) (at 101.8414 112.014 0)
       (effects (font (size 1.27 1.27)) (justify left))
     )
@@
       (effects (font (size 1.27 1.27)) (justify left))
     )
-    (property "Footprint" "" (id 2) (at 99.822 132.08 0)
+    (property "Footprint" "Package_DIP:DIP-20_W7.62mm_Socket_LongPads" (id 2) (at 99.822 132.08 0)
       (effects (font (size 1.27 1.27)) hide)
     )
@@
   (symbol (lib_id "74xx:74LS139") (at 41.656 82.296 0) (unit 3)
     (in_bom yes) (on_board yes) (fields_autoplaced)
-    (property "Reference" "U?" (id 0) (at 48.26 81.0259 0)
+    (property "Reference" "U8" (id 0) (at 48.26 81.0259 0)
       (effects (font (size 1.27 1.27)) (justify left))
     )
@@
       (effects (font (size 1.27 1.27)) (justify left))
     )
-    (property "Footprint" "" (id 2) (at 41.656 82.296 0)
+    (property "Footprint" "Package_DIP:DIP-16_W7.62mm_Socket_LongPads" (id 2) (at 41.656 82.296 0)
       (effects (font (size 1.27 1.27)) hide)
     )
@@
   (symbol (lib_id "74xx:74LS377") (at 99.822 42.926 0) (unit 1)
     (in_bom yes) (on_board yes) (fields_autoplaced)
-    (property "Reference" "U?" (id 0) (at 101.8414 22.86 0)
+    (property "Reference" "U9" (id 0) (at 101.8414 22.86 0)
       (effects (font (size 1.27 1.27)) (justify left))
     )
@@
       (effects (font (size 1.27 1.27)) (justify left))
     )
-    (property "Footprint" "" (id 2) (at 99.822 42.926 0)
+    (property "Footprint" "Package_DIP:DIP-20_W7.62mm_Socket_LongPads" (id 2) (at 99.822 42.926 0)
       (effects (font (size 1.27 1.27)) hide)
     )
@@
   (symbol (lib_id "74xx:74LS377") (at 99.822 87.884 0) (unit 1)
     (in_bom yes) (on_board yes) (fields_autoplaced)
-    (property "Reference" "U?" (id 0) (at 101.8414 67.818 0)
+    (property "Reference" "U10" (id 0) (at 101.8414 67.818 0)
       (effects (font (size 1.27 1.27)) (justify left))
     )
@@
       (effects (font (size 1.27 1.27)) (justify left))
     )
-    (property "Footprint" "" (id 2) (at 99.822 87.884 0)
+    (property "Footprint" "Package_DIP:DIP-20_W7.62mm_Socket_LongPads" (id 2) (at 99.822 87.884 0)
       (effects (font (size 1.27 1.27)) hide)
     )
@@
   (symbol (lib_id "power:VCC") (at 41.656 69.596 0) (unit 1)
     (in_bom yes) (on_board yes) (fields_autoplaced)
-    (property "Reference" "#PWR?" (id 0) (at 41.656 73.406 0)
+    (property "Reference" "#PWR0125" (id 0) (at 41.656 73.406 0)
       (effects (font (size 1.27 1.27)) hide)
     )
@@
   (symbol (lib_id "74xx:74LS139") (at 41.91 39.116 0) (unit 1)
     (in_bom yes) (on_board yes) (fields_autoplaced)
-    (property "Reference" "U?" (id 0) (at 41.91 29.21 0))
+    (property "Reference" "U8" (id 0) (at 41.91 29.21 0))
     (property "Value" "74LS139" (id 1) (at 41.91 31.75 0))
-    (property "Footprint" "" (id 2) (at 41.91 39.116 0)
+    (property "Footprint" "Package_DIP:DIP-16_W7.62mm_Socket_LongPads" (id 2) (at 41.91 39.116 0)
       (effects (font (size 1.27 1.27)) hide)
     )
@@
   (symbol (lib_id "power:GND") (at 102.87 152.4 0) (unit 1)
     (in_bom yes) (on_board yes) (fields_autoplaced)
-    (property "Reference" "#PWR?" (id 0) (at 102.87 158.75 0)
+    (property "Reference" "#PWR0126" (id 0) (at 102.87 158.75 0)
       (effects (font (size 1.27 1.27)) hide)
     )
@@
   (symbol (lib_id "power:VCC") (at 120.396 22.606 0) (unit 1)
     (in_bom yes) (on_board yes) (fields_autoplaced)
-    (property "Reference" "#PWR?" (id 0) (at 120.396 26.416 0)
+    (property "Reference" "#PWR0123" (id 0) (at 120.396 26.416 0)
       (effects (font (size 1.27 1.27)) hide)
     )
