File: Hardware/Schematics/PC_SP_IR_Selector/PC_SP_IR_Selector.kicad_pcb (KiCad board)
At the start: 2 copper layers, 89.3 x 101.3 mm, 17 parts, among them J1 Conn_01x05, J2 Conn_01x10, J3 Conn_01x10, J4 Conn_01x10, J5 Conn_01x10, J6 Conn_01x10, J7 Conn_01x10, J8 Conn_01x10, J9 Conn_01x10, U1 74LS08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

Commit message: Boards Done
Parts:
- J2: footprint Connector_PinSocket_2.54mm:PinSocket_1x10_P2.54mm_Vertical -> Connector_PinSocket_2.54mm:PinSocket_1x05_P2.54mm_Vertical
- U2: footprint Package_DIP:DIP-16_W7.62mm_Socket_LongPads -> Package_DIP:DIP-14_W7.62mm_Socket_LongPads
