File: Hardware/Schematics/Register/Register.kicad_pcb (KiCad board)
At the start: 2 copper layers, 55.7 x 41.5 mm, 13 parts, among them J1 Conn_02x15_Counter_Clockwise, U1 74LS377, U2 74LS245, U3 74LS245

Commit message: Boards Done
Other:
- board text added: "Designed By: Alex Dasneves"
Changed lines of the file:
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@@
   )
   (gr_rect (start 32.23 53.49) (end 87.96 94.99) (layer "Edge.Cuts") (width 0.1) (fill none))
+  (gr_text "Designed By:\nAlex Dasneves" (at 36.322 80.772 90) (layer "F.SilkS")
+    (effects (font (size 1 1) (thickness 0.15)))
+  )
   (segment (start 48.1252 57.8651) (end 46.6051 56.345) (width 0.25) (layer "F.Cu") (net 1))
   (segment (start 50.98 57.8651) (end 48.1252 57.8651) (width 0.25) (layer "F.Cu") (net 1))
