File: Hardware/Schematics/Registers/Registers.kicad_pcb (KiCad board)
At the start: 4 copper layers, 91 parts, among them J1 Conn_01x19, J2 Conn_01x08, J3 Conn_01x08, U1 74LS139, U10 74LS245, U11 74LS245, U12 74LS245, U13 74LS245, U14 74LS245, U15 74LS245, U16 74LS245, U2 74LS139, U3 74LS377, U5 74LS377, U7 74LS377, U8 74LS377, U9 74LS245

Commit message: Updated Schematics
Parts:
- removed C1, C10, C11, C12, C13, C14, C15, C16, C2, C3, C4, C5, C6, C7, C8, C9: C, Capacitor_THT:C_Rect_L9.0mm_W2.5mm_P7.50mm_MKT
- removed D1, D10, D11, D12, D13, D14, D15, D16, D17, D18, D19, D2, D20, D21, D22, D23, D24, D25, D26, D27, D28, D29, D3, D30, D31, D32, D33, D34, D35, D36, D37, D38, D39, D4, D40, D41, D42, D43, D44, D45, D46, D47, D48, D5, D6, D7, D8, D9: LED, LED_THT:LED_D3.0mm
- removed RD1, RS1, U5, U7, U8: 74LS377, Package_DIP:DIP-20_W7.62mm_LongPads
- removed REF** (x2): MountingHole_5.5mm, MountingHole:MountingHole_5.5mm
- removed RN1, RN2, RN3, RN4, RN5, RN6: R_Network08, Resistor_THT:R_Array_SIP9
- removed U10, U11, U12, U13, U14, U15, U16, U9: 74LS245, Package_DIP:DIP-20_W7.62mm_LongPads
- added J4: Conn_02x15_Counter_Clockwise, Connector_PinHeader_2.54mm:PinHeader_2x15_P2.54mm_Vertical, F.Cu at (72.7, 21.6)
- added J5: Conn_02x15_Counter_Clockwise, Connector_PinHeader_2.54mm:PinHeader_2x15_P2.54mm_Vertical, F.Cu at (58.9, 21.6)
- added J6: Conn_02x15_Counter_Clockwise, Connector_PinHeader_2.54mm:PinHeader_2x15_P2.54mm_Vertical, F.Cu at (86.4, 21.6)
- added J7: Conn_01x10, Connector_PinHeader_2.54mm:PinHeader_1x10_P2.54mm_Vertical, F.Cu at (111.7, 21.4)
- added J8: Conn_01x10, Connector_PinHeader_2.54mm:PinHeader_1x10_P2.54mm_Vertical, F.Cu at (111.2, 51.1)
- added U4: 74LS377, Package_DIP:DIP-20_W7.62mm_Socket_LongPads, F.Cu at (94.6, 51.3)
- J1: value Conn_01x19 -> Conn_02x05_Counter_Clockwise; footprint Connector_PinHeader_2.54mm:PinHeader_1x19_P2.54mm_Vertical -> Connector_PinHeader_2.54mm:PinHeader_2x05_P2.54mm_Vertical
- J2: value Conn_01x08 -> Conn_01x10
- J3: value Conn_01x08 -> Conn_02x15_Counter_Clockwise; footprint Connector_PinHeader_2.54mm:PinHeader_1x10_P2.54mm_Vertical -> Connector_PinHeader_2.54mm:PinHeader_2x15_P2.54mm_Vertical
- U1, U2: footprint Package_DIP:DIP-16_W7.62mm_LongPads -> Package_DIP:DIP-16_W7.62mm_Socket_LongPads
- U3: footprint Package_DIP:DIP-20_W7.62mm_LongPads -> Package_DIP:DIP-20_W7.62mm_Socket_LongPads
- moved J3 101.9 mm to (45.1, 21.7), turned to 0 degrees
- moved U2 70.3 mm to (71.1, 73.6), turned to 90 degrees
- moved J2 70.1 mm to (19.8, 44.6), turned to 180 degrees
- moved U3 67.4 mm to (95.0, 21.7), turned to 0 degrees
- moved U1 44.9 mm to (39.7, 73.0), turned to 90 degrees
- moved J1 40.2 mm to (20.6, 56.1)
Connections:
- J1 pad 1: GND -> VCC
- J1 pad 10: Net-(U3-Pad18) -> Net-(J1-Pad10)
- J1 pad 2: VCC -> Net-(J1-Pad2)
- J1 pad 3: Net-(U3-Pad3) -> Net-(J1-Pad3)
- J1 pad 5: Net-(J1-Pad5) -> /CLK
- J1 pad 6: Net-(J1-Pad6) -> GND
- J2 pad 2: Net-(D16-Pad2) -> /D_{7}
- J2 pad 3: Net-(D15-Pad2) -> /D_{6}
- J2 pad 4: Net-(D14-Pad2) -> /D_{5}
- J2 pad 5: Net-(D12-Pad2) -> /D_{4}
- J2 pad 6: Net-(D10-Pad2) -> /D_{3}
- J2 pad 7: Net-(D8-Pad2) -> /D_{2}
- J2 pad 8: Net-(D6-Pad2) -> /D_{1}
- J2 pad 9: Net-(D4-Pad2) -> /D_{0}
- J3 pad 1: GND -> VCC
- J3 pad 10: VCC -> /RD_{4}
- J3 pad 2: Net-(D37-Pad2) -> /RD_{0}
- J3 pad 3: Net-(D35-Pad2) -> /D_{0}
- J3 pad 4: Net-(D33-Pad2) -> /RD_{1}
- J3 pad 5: Net-(D31-Pad2) -> /D_{1}
- J3 pad 6: Net-(D29-Pad2) -> /RD_{2}
- J3 pad 7: Net-(D27-Pad2) -> /D_{2}
- J3 pad 8: Net-(D26-Pad2) -> /RD_{3}
- J3 pad 9: Net-(D25-Pad2) -> /D_{3}
- U1 pad 1: Net-(J1-Pad13) -> Net-(J1-Pad2)
- U1 pad 10: /RD_{SelectX} -> Net-(J5-Pad23)
- U1 pad 11: /RD_{SelectB} -> Net-(J4-Pad23)
- U1 pad 12: /RD_{SelectA} -> Net-(J3-Pad23)
- U1 pad 13: Net-(J1-Pad14) -> Net-(J1-Pad10)
- U1 pad 14: Net-(J1-Pad15) -> Net-(J1-Pad9)
- U1 pad 15: Net-(J1-Pad16) -> Net-(J1-Pad3)
- U1 pad 2: Net-(J1-Pad12) -> Net-(J1-Pad9)
- U1 pad 3: Net-(J1-Pad11) -> Net-(J1-Pad10)
- U1 pad 4: /RS_{SelectA} -> Net-(J3-Pad21)
- U1 pad 5: /RS_{SelectB} -> Net-(J4-Pad21)
- U1 pad 6: /RS_{SelectX} -> Net-(J5-Pad21)
- U1 pad 7: /RS_{SelectY} -> Net-(J6-Pad21)
- U1 pad 9: /RD_{SelectY} -> Net-(J6-Pad23)
- U2 pad 1: Net-(J1-Pad19) -> Net-(J1-Pad4)
- U2 pad 10: unconnected-(U2-Pad10) -> (no net)
- U2 pad 11: unconnected-(U2-Pad11) -> (no net)
- U2 pad 12: unconnected-(U2-Pad12) -> (no net)
- U2 pad 13: unconnected-(U2-Pad13) -> (no net)
- U2 pad 14: unconnected-(U2-Pad14) -> (no net)
- U2 pad 15: unconnected-(U2-Pad15) -> (no net)
- U2 pad 2: Net-(J1-Pad18) -> Net-(J1-Pad7)
- U2 pad 3: Net-(J1-Pad17) -> Net-(J1-Pad8)
- U2 pad 4: Net-(U2-Pad4) -> Net-(J3-Pad25)
- U2 pad 9: unconnected-(U2-Pad9) -> (no net)
- U3 pad 1: Net-(U2-Pad4) -> Net-(J1-Pad3)
- U3 pad 11: Net-(U3-Pad11) -> /CLK
- U3 pad 13: Net-(J1-Pad7) -> /RD_{4}
- U3 pad 14: Net-(J1-Pad8) -> /RD_{5}
- U3 pad 17: Net-(J1-Pad9) -> /RD_{6}
- U3 pad 18: Net-(U3-Pad18) -> /RD_{7}
- U3 pad 3: Net-(U3-Pad3) -> /RD_{0}
- U3 pad 4: Net-(J1-Pad4) -> /RD_{1}
- U3 pad 7: Net-(J1-Pad5) -> /RD_{2}
- U3 pad 8: Net-(J1-Pad6) -> /RD_{3}
Routing:
- net GND: track 689.1 -> 198.6 mm
- net VCC: track 539.5 -> 231.4 mm
- net Net-(D4-Pad2): track 235.7 -> 0.00 mm
- net Net-(D16-Pad2): track 226.8 -> 0.00 mm
- net Net-(D6-Pad2): track 224.4 -> 0.00 mm
- net Net-(D8-Pad2): track 220.7 -> 0.00 mm
- net Net-(D15-Pad2): track 216.9 -> 0.00 mm
- net Net-(D14-Pad2): track 215.8 -> 0.00 mm
- net Net-(D10-Pad2): track 213.6 -> 0.00 mm
- net Net-(D12-Pad2): track 211.2 -> 0.00 mm
- net Net-(J1-Pad18): track 199.0 -> 0.00 mm
- net Net-(J1-Pad19): track 197.8 -> 0.00 mm
- net Net-(J1-Pad17): track 197.7 -> 0.00 mm
- net Net-(D34-Pad2): track 174.5 -> 0.00 mm
- net Net-(D39-Pad2): track 166.5 -> 0.00 mm
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- removed copper zone on B.Cu, net GND
- removed copper zone on F.Cu, net GND
Other:
- board outline added: 96.9 x 58.9 mm
- copper layers 4 -> 2

Commit message: Boards Done
Other:
- board text added: "Designed by: Alex Dasneves"
Changed lines of the file:
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@@
   )
   (gr_rect (start 17.43 18.17) (end 114.38 77.06) (layer "Edge.Cuts") (width 0.1) (fill none))
+  (gr_text "Designed by:\nAlex Dasneves" (at 23.622 74.93) (layer "F.SilkS")
+    (effects (font (size 1 1) (thickness 0.15)))
+  )
   (segment (start 111.18 51.135) (end 103.9401 51.135) (width 0.25) (layer "F.Cu") (net 1))
   (segment (start 85.8125 21.65) (end 86.3892 21.65) (width 0.25) (layer "F.Cu") (net 1))
